File: ModuleBattery18650.kicad_sch (KiCad schematic)
At the start: 26 parts, among them J1 Connector_2p, J2 Connector_2p_r, T1 SISH615ADN, T2 SISH615ADN, T3 FDN337N, T4 SISH615ADN, T5 SISH615ADN, U1 MCP121T-315E

Commit message: rev00
Parts:
- added D1: LED, 0ESN_Lib:D_0603_1608Metric_Pad1.05x0.95mm_HandSolder, symbol 0ESN_Lib:LED
- added R4: 150R, Resistor_SMD:R_0805_2012Metric_Pad1.20x1.40mm_HandSolder, symbol 0ESN_Lib:R
- JP1: footprint 0ESN_Lib:PinHeader_1x02_P1.27mm_Vertical -> Jumper:SolderJumper-2_P1.3mm_Open_RoundedPad1.0x1.5mm
- R1, R2, R3, RS1, RS2: footprint 0ESN_Lib:R_0603_1608Metric_Pad0.98x0.95mm_HandSolder -> Resistor_SMD:R_0603_1608Metric_Pad0.98x0.95mm_HandSolder
- T3: symbol 0l2:MOSFET-N -> 0ESN_Lib:FDN337N
Connections:
- net GND: now also R4.2
- net at JP1.2 (B), R1.1, T1.3 (D)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: now also D1.1 (A)
- new net: D1.2 (K), R4.1
Changed lines of the file:
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@@
+    (stroke (width 0) (type default) (color 0 0 0 0))
+  )
+  (wire (pts (xy 69.85 80.01) (xy 69.85 83.82))
     (stroke (width 0) (type default) (color 0 0 0 0))
   )
@@
     (stroke (width 0) (type default) (color 0 0 0 0))
   )
+  (wire (pts (xy 69.85 58.42) (xy 69.85 62.23))
+    (stroke (width 0) (type default) (color 0 0 0 0))
+  )
   (polyline (pts (xy 175.26 34.29) (xy 236.22 34.29))
     (stroke (width 0) (type default) (color 0 0 0 0))
@@
   )
   (wire (pts (xy 106.68 83.82) (xy 106.68 67.31))
+    (stroke (width 0) (type default) (color 0 0 0 0))
+  )
+  (wire (pts (xy 69.85 69.85) (xy 69.85 72.39))
     (stroke (width 0) (type default) (color 0 0 0 0))
   )
@@
     (property "Reference" "RS1" (id 0) (at 151.13 71.6264 90))
     (property "Value" "0R NP" (id 1) (at 151.13 74.1633 90))
-    (property "Footprint" "0ESN_Lib:R_0603_1608Metric_Pad0.98x0.95mm_HandSolder" (id 2) (at 151.13 70.358 90)
+    (property "Footprint" "Resistor_SMD:R_0603_1608Metric_Pad0.98x0.95mm_HandSolder" (id 2) (at 151.13 70.358 90)
       (effects (font (size 1.27 1.27)) hide)
     )
@@
       (effects (font (size 1.27 1.27)) hide)
     )
-    (property "Footprint" "0ESN_Lib:PinHeader_1x02_P1.27mm_Vertical" (id 2) (at 58.42 58.42 0)
+    (property "Footprint" "Jumper:SolderJumper-2_P1.3mm_Open_RoundedPad1.0x1.5mm" (id 2) (at 58.42 58.42 0)
       (effects (font (size 1.27 1.27)) hide)
     )
@@
     (pin "2")
   )
-  (symbol (lib_id "0l2:MOSFET-N") (at 215.9 77.47 270) (unit 1)
+  (symbol (lib_id "0ESN_Lib:FDN337N") (at 215.9 77.47 270) (unit 1)
     (in_bom yes) (on_board yes) (fields_autoplaced)
     (property "Reference" "T3" (id 0) (at 219.075 76.4938 90)
@@
     (pin "1")
   )
+  (symbol (lib_id "power:GND") (at 69.85 83.82 0) (unit 1)
+    (in_bom yes) (on_board yes) (fields_autoplaced)
+    (property "Reference" "#PWR010" (id 0) (at 69.85 90.17 0)
+      (effects (font (size 1.27 1.27)) hide)
+    )
+    (property "Value" "GND" (id 1) (at 69.85 88.2634 0))
+    (property "Footprint" "" (id 2) (at 69.85 83.82 0)
+      (effects (font (size 1.27 1.27)) hide)
+    )
+    (property "Datasheet" "" (id 3) (at 69.85 83.82 0)
+      (effects (font (size 1.27 1.27)) hide)
+    )
+    (pin "1")
+  )
   (symbol (lib_id "power:GND") (at 106.68 83.82 0) (unit 1)
     (in_bom yes) (on_board yes) (fields_autoplaced)
@@
       (effects (font (size 1.27 1.27)) (justify left))
     )
-    (property "Footprint" "0ESN_Lib:R_0603_1608Metric_Pad0.98x0.95mm_HandSolder" (id 2) (at 139.192 72.39 90)
+    (property "Footprint" "Resistor_SMD:R_0603_1608Metric_Pad0.98x0.95mm_HandSolder" (id 2) (at 139.192 72.39 90)
       (effects (font (size 1.27 1.27)) hide)
     )
@@
     (pin "3")
   )
+  (symbol (lib_id "0ESN_Lib:LED") (at 69.85 66.04 270) (unit 1)
+    (in_bom yes) (on_board yes) (fields_autoplaced)
+    (property "Reference" "D1" (id 0) (at 71.882 66.7928 90)
+      (effects (font (size 1.27 1.27)) (justify left))
+    )
+    (property "Value" "LED" (id 1) (at 71.882 69.3297 90)
+      (effects (font (size 1.27 1.27)) (justify left))
+    )
+    (property "Footprint" "0ESN_Lib:D_0603_1608Metric_Pad1.05x0.95mm_HandSolder" (id 2) (at 74.168 68.58 0)
+      (effects (font (size 1.27 1.27)) hide)
+    )
+    (property "Datasheet" "~" (id 3) (at 69.85 66.04 0)
+      (effects (font (size 1.27 1.27)) hide)
+    )
+    (pin "1")
+    (pin "2")
+  )
+  (symbol (lib_id "0ESN_Lib:R") (at 69.85 76.2 0) (unit 1)
+    (in_bom yes) (on_board yes) (fields_autoplaced)
+    (property "Reference" "R4" (id 0) (at 71.628 75.3653 0)
+      (effects (font (size 1.27 1.27)) (justify left))
+    )
+    (property "Value" "150R" (id 1) (at 71.628 77.9022 0)
+      (effects (font (size 1.27 1.27)) (justify left))
+    )
+    (property "Footprint" "Resistor_SMD:R_0805_2012Metric_Pad1.20x1.40mm_HandSolder" (id 2) (at 68.072 76.2 90)
+      (effects (font (size 1.27 1.27)) hide)
+    )
+    (property "Datasheet" "~" (id 3) (at 69.85 76.2 0)
+      (effects (font (size 1.27 1.27)) hide)
+    )
+    (pin "1")
+    (pin "2")
+  )
   (symbol (lib_id "Device:R") (at 208.28 64.77 0) (unit 1)
     (in_bom yes) (on_board yes) (fields_autoplaced)
@@
       (effects (font (size 1.27 1.27)) (justify left))
     )
-    (property "Footprint" "0ESN_Lib:R_0603_1608Metric_Pad0.98x0.95mm_HandSolder" (id 2) (at 206.502 64.77 90)
+    (property "Footprint" "Resistor_SMD:R_0603_1608Metric_Pad0.98x0.95mm_HandSolder" (id 2) (at 206.502 64.77 90)
       (effects (font (size 1.27 1.27)) hide)
     )
@@
     (property "Reference" "RS2" (id 0) (at 214.63 43.5442 90))
     (property "Value" "0R NP" (id 1) (at 214.63 46.0811 90))
-    (property "Footprint" "0ESN_Lib:R_0603_1608Metric_Pad0.98x0.95mm_HandSolder" (id 2) (at 214.63 50.038 90)
+    (property "Footprint" "Resistor_SMD:R_0603_1608Metric_Pad0.98x0.95mm_HandSolder" (id 2) (at 214.63 50.038 90)
       (effects (font (size 1.27 1.27)) hide)
     )
@@
       (effects (font (size 1.27 1.27)) (justify left))
     )
-    (property "Footprint" "0ESN_Lib:R_0603_1608Metric_Pad0.98x0.95mm_HandSolder" (id 2) (at 198.882 64.77 90)
+    (property "Footprint" "Resistor_SMD:R_0603_1608Metric_Pad0.98x0.95mm_HandSolder" (id 2) (at 198.882 64.77 90)
       (effects (font (size 1.27 1.27)) hide)
     )
@@
       (reference "#PWR09") (unit 1) (value "GND") (footprint "")
     )
+    (path "/86fbcd37-0120-4038-acee-2c118f1ca0df"
+      (reference "#PWR010") (unit 1) (value "GND") (footprint "")
+    )
     (path "/3563b52b-d2c0-41b9-aeca-2af682e9e33e"
       (reference "BT1") (unit 1) (value "LiIon 3.7V 4.2V") (footprint "0ESN_Lib:18650_Battery_holder")
@@
       (reference "C1") (unit 1) (value "4.7uF") (footprint "0ESN_Lib:C_0805_2012Metric_Pad1.18x1.45mm_HandSolder")
     )
+    (path "/a8709592-4597-4538-8554-191b10919da4"
+      (reference "D1") (unit 1) (value "LED") (footprint "0ESN_Lib:D_0603_1608Metric_Pad1.05x0.95mm_HandSolder")
+    )
     (path "/05911fbb-7eaf-441b-a6f2-e9dd11e758e0"
       (reference "F1") (unit 1) (value "xx mA") (footprint "0ESN_Lib:Fuse_1206_3216Metric_Pad1.42x1.75mm_HandSolder")
@@
     )
     (path "/18962da5-7338-4528-bbd2-01ad0e636188"
-      (reference "JP1") (unit 1) (value "Jumper_2_Bridged") (footprint "0ESN_Lib:PinHeader_1x02_P1.27mm_Vertical")
+      (reference "JP1") (unit 1) (value "Jumper_2_Bridged") (footprint "Jumper:SolderJumper-2_P1.3mm_Open_RoundedPad1.0x1.5mm")
     )
     (path "/a320823e-63fc-45b5-8cb1-0bb20ad43df5"
-      (reference "R1") (unit 1) (value "1M") (footprint "0ESN_Lib:R_0603_1608Metric_Pad0.98x0.95mm_HandSolder")
+      (reference "R1") (unit 1) (value "1M") (footprint "Resistor_SMD:R_0603_1608Metric_Pad0.98x0.95mm_HandSolder")
     )
     (path "/dae82fe2-b96e-47e4-9b90-8bedaaf1bdf2"
-      (reference "R2") (unit 1) (value "1M") (footprint "0ESN_Lib:R_0603_1608Metric_Pad0.98x0.95mm_HandSolder")
+      (reference "R2") (unit 1) (value "1M") (footprint "Resistor_SMD:R_0603_1608Metric_Pad0.98x0.95mm_HandSolder")
     )
     (path "/b8aa7f13-7acf-4e93-85dd-3239f8cbdd45"
-      (reference "R3") (unit 1) (value "1M") (footprint "0ESN_Lib:R_0603_1608Metric_Pad0.98x0.95mm_HandSolder")
+      (reference "R3") (unit 1) (value "1M") (footprint "Resistor_SMD:R_0603_1608Metric_Pad0.98x0.95mm_HandSolder")
+    )
+    (path "/b87c2113-bcfe-4f97-8a57-cb58b7f60e46"
+      (reference "R4") (unit 1) (value "150R") (footprint "Resistor_SMD:R_0805_2012Metric_Pad1.20x1.40mm_HandSolder")
     )
     (path "/0d535591-7c94-4bcb-ab85-6f82a5cb2691"
-      (reference "RS1") (unit 1) (value "0R NP") (footprint "0ESN_Lib:R_0603_1608Metric_Pad0.98x0.95mm_HandSolder")
+      (reference "RS1") (unit 1) (value "0R NP") (footprint "Resistor_SMD:R_0603_1608Metric_Pad0.98x0.95mm_HandSolder")
     )
     (path "/d96ba3bc-bbbe-4e7c-b19a-e66455ec7e04"
-      (reference "RS2") (unit 1) (value "0R NP") (footprint "0ESN_Lib:R_0603_1608Metric_Pad0.98x0.95mm_HandSolder")
+      (reference "RS2") (unit 1) (value "0R NP") (footprint "Resistor_SMD:R_0603_1608Metric_Pad0.98x0.95mm_HandSolder")
     )
     (path "/1faa3af5-61f3-4f40-a3ca-42ba69cf237c"

Commit message: revision 01
Parts:
- C1: footprint 0ESN_Lib:C_0805_2012Metric_Pad1.18x1.45mm_HandSolder -> Capacitor_SMD:C_0805_2012Metric_Pad1.18x1.45mm_HandSolder
- D1: footprint 0ESN_Lib:D_0603_1608Metric_Pad1.05x0.95mm_HandSolder -> Diode_SMD:D_0603_1608Metric_Pad1.05x0.95mm_HandSolder
Connections:
- net GND: now also T1.4 (G), T5.4 (G); no longer T1.1 (G), T5.1 (G)
- net Vbat: now also T5.1 (S), T5.3 (S)
- net at C1.1, F1.2, RS1.1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: now also T1.1 (S), T1.3 (S), T2.1 (S), T2.3 (S)
- net at R2.1, R3.1, RS1.2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: now also T2.5 (D), T4.1 (S), T4.3 (S); no longer T2.3 (D)
- net at D1.1 (A), JP1.2 (B), R1.1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: now also T1.5 (D), T2.4 (G); no longer T1.3 (D), T2.1 (G)
- net at RS2.2, TP8.1: now also T4.5 (D), T5.5 (D); no longer T4.3 (D), T5.3 (D)
- net at R3.2, T3.3 (D), TP7.1: now also T4.4 (G); no longer T4.1 (G)
Changed lines of the file:
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@@
     (pin "1")
   )
-  (symbol (lib_name "SISH615ADN_3") (lib_id "0ESN_Lib:SISH615ADN") (at 91.44 58.42 0) (unit 1)
+  (symbol (lib_id "0ESN_Lib:SISH615ADN") (at 91.44 58.42 0) (unit 1)
     (in_bom yes) (on_board yes) (fields_autoplaced)
     (property "Reference" "T1" (id 0) (at 91.44 51.7959 0)
@@
     (pin "2")
     (pin "3")
+    (pin "4")
+    (pin "5")
   )
   (symbol (lib_id "power:GND") (at 93.98 83.82 0) (unit 1)
@@
     (pin "1")
   )
-  (symbol (lib_name "SISH615ADN_1") (lib_id "0ESN_Lib:SISH615ADN") (at 151.13 58.42 180) (unit 1)
+  (symbol (lib_id "0ESN_Lib:SISH615ADN") (at 151.13 58.42 180) (unit 1)
     (in_bom yes) (on_board yes)
     (property "Reference" "T2" (id 0) (at 154.94 50.8 0)
@@
     (pin "2")
     (pin "3")
+    (pin "4")
+    (pin "5")
   )
   (symbol (lib_id "Device:Battery_Cell") (at 118.11 76.2 0) (unit 1)
@@
     (pin "1")
   )
-  (symbol (lib_name "TestPoint_3") (lib_id "0ESN_Lib:TestPoint") (at 260.35 58.42 0) (unit 1)
+  (symbol (lib_id "0ESN_Lib:TestPoint") (at 260.35 58.42 0) (unit 1)
     (in_bom yes) (on_board yes) (fields_autoplaced)
     (property "Reference" "TP9" (id 0) (at 260.35 53.34 0))
@@
     (pin "1")
   )
-  (symbol (lib_name "SISH615ADN_2") (lib_id "0ESN_Lib:SISH615ADN") (at 247.65 58.42 0) (unit 1)
+  (symbol (lib_id "0ESN_Lib:SISH615ADN") (at 247.65 58.42 0) (unit 1)
     (in_bom yes) (on_board yes) (fields_autoplaced)
     (property "Reference" "T5" (id 0) (at 247.65 51.7959 0)
@@
     (pin "2")
     (pin "3")
+    (pin "4")
+    (pin "5")
   )
   (symbol (lib_id "0ESN_Lib:TestPoint") (at 78.74 58.42 0) (unit 1)
@@
     (pin "1")
   )
-  (symbol (lib_name "TestPoint_5") (lib_id "0ESN_Lib:TestPoint") (at 204.47 80.01 0) (unit 1)
+  (symbol (lib_id "0ESN_Lib:TestPoint") (at 204.47 80.01 0) (unit 1)
     (in_bom yes) (on_board yes) (fields_autoplaced)
     (property "Reference" "TP6" (id 0) (at 204.47 74.93 0))
@@
     (pin "2")
   )
-  (symbol (lib_name "TestPoint_4") (lib_id "0ESN_Lib:TestPoint") (at 227.33 68.58 0) (unit 1)
+  (symbol (lib_id "0ESN_Lib:TestPoint") (at 227.33 68.58 0) (unit 1)
     (in_bom yes) (on_board yes) (fields_autoplaced)
     (property "Reference" "TP7" (id 0) (at 227.33 63.5 0))
@@
       (effects (font (size 1.27 1.27)) (justify left))
     )
-    (property "Footprint" "0ESN_Lib:D_0603_1608Metric_Pad1.05x0.95mm_HandSolder" (id 2) (at 74.168 68.58 0)
+    (property "Footprint" "Diode_SMD:D_0603_1608Metric_Pad1.05x0.95mm_HandSolder" (id 2) (at 74.168 68.58 0)
       (effects (font (size 1.27 1.27)) hide)
     )
@@
     (pin "2")
   )
-  (symbol (lib_name "TestPoint_3") (lib_id "0ESN_Lib:TestPoint") (at 233.68 58.42 0) (unit 1)
+  (symbol (lib_id "0ESN_Lib:TestPoint") (at 233.68 58.42 0) (unit 1)
     (in_bom yes) (on_board yes) (fields_autoplaced)
     (property "Reference" "TP8" (id 0) (at 233.68 53.34 0))
@@
       (effects (font (size 1.27 1.27)) (justify left))
     )
-    (property "Footprint" "0ESN_Lib:C_0805_2012Metric_Pad1.18x1.45mm_HandSolder" (id 2) (at 107.6452 67.31 0)
+    (property "Footprint" "Capacitor_SMD:C_0805_2012Metric_Pad1.18x1.45mm_HandSolder" (id 2) (at 107.6452 67.31 0)
       (effects (font (size 1.27 1.27)) hide)
     )
@@
     (pin "2")
     (pin "3")
-  )
-  (symbol (lib_name "TestPoint_1") (lib_id "0ESN_Lib:TestPoint") (at 46.99 58.42 0) (unit 1)
+    (pin "4")
+    (pin "5")
+  )
+  (symbol (lib_id "0ESN_Lib:TestPoint") (at 46.99 58.42 0) (unit 1)
     (in_bom yes) (on_board yes) (fields_autoplaced)
     (property "Reference" "TP1" (id 0) (at 46.99 53.34 0))
@@
     )
     (path "/d48cd143-8b88-4905-bfb8-0024c83d29a0"
-      (reference "C1") (unit 1) (value "4.7uF") (footprint "0ESN_Lib:C_0805_2012Metric_Pad1.18x1.45mm_HandSolder")
+      (reference "C1") (unit 1) (value "4.7uF") (footprint "Capacitor_SMD:C_0805_2012Metric_Pad1.18x1.45mm_HandSolder")
     )
     (path "/a8709592-4597-4538-8554-191b10919da4"
-      (reference "D1") (unit 1) (value "LED") (footprint "0ESN_Lib:D_0603_1608Metric_Pad1.05x0.95mm_HandSolder")
+      (reference "D1") (unit 1) (value "LED") (footprint "Diode_SMD:D_0603_1608Metric_Pad1.05x0.95mm_HandSolder")
     )
     (path "/05911fbb-7eaf-441b-a6f2-e9dd11e758e0"

Commit message: ^small changes
Parts:
- added H1, H2, H3: MountingHole, MountingHole:MountingHole_4.3mm_M4, symbol Mechanical:MountingHole
Changed lines of the file:
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@@
 (kicad_sch (version 20211123) (generator eeschema)
   (paper "A4")
-  (junction (at 156.21 58.42) (diameter 0) (color 0 0 0 0)
-  )
   (junction (at 143.51 58.42) (diameter 0) (color 0 0 0 0)
   )
@@
   )
   (polyline (pts (xy 256.54 66.04) (xy 256.54 49.53))
-    (stroke (width 0) (type default) (color 0 0 0 0))
-  )
-  (wire (pts (xy 153.67 58.42) (xy 156.21 58.42))
     (stroke (width 0) (type default) (color 0 0 0 0))
   )
@@
     (pin "1")
   )
+  (symbol (lib_id "Mechanical:MountingHole") (at 36.83 29.21 0) (unit 1)
+    (in_bom yes) (on_board yes) (fields_autoplaced)
+    (property "Reference" "H2" (id 0) (at 39.37 27.9399 0)
+      (effects (font (size 1.27 1.27)) (justify left))
+    )
+    (property "Value" "MountingHole" (id 1) (at 39.37 30.4799 0)
+      (effects (font (size 1.27 1.27)) (justify left))
+    )
+    (property "Footprint" "MountingHole:MountingHole_4.3mm_M4" (id 2) (at 36.83 29.21 0)
+      (effects (font (size 1.27 1.27)) hide)
+    )
+    (property "Datasheet" "~" (id 3) (at 36.83 29.21 0)
+      (effects (font (size 1.27 1.27)) hide)
+    )
+  )
   (symbol (lib_id "0ESN_Lib:SISH615ADN") (at 151.13 58.42 180) (unit 1)
     (in_bom yes) (on_board yes)
@@
     (pin "2")
   )
+  (symbol (lib_id "Mechanical:MountingHole") (at 36.83 34.29 0) (unit 1)
+    (in_bom yes) (on_board yes) (fields_autoplaced)
+    (property "Reference" "H3" (id 0) (at 39.37 33.0199 0)
+      (effects (font (size 1.27 1.27)) (justify left))
+    )
+    (property "Value" "MountingHole" (id 1) (at 39.37 35.5599 0)
+      (effects (font (size 1.27 1.27)) (justify left))
+    )
+    (property "Footprint" "MountingHole:MountingHole_4.3mm_M4" (id 2) (at 36.83 34.29 0)
+      (effects (font (size 1.27 1.27)) hide)
+    )
+    (property "Datasheet" "~" (id 3) (at 36.83 34.29 0)
+      (effects (font (size 1.27 1.27)) hide)
+    )
+  )
+  (symbol (lib_id "Mechanical:MountingHole") (at 36.83 24.13 0) (unit 1)
+    (in_bom yes) (on_board yes) (fields_autoplaced)
+    (property "Reference" "H1" (id 0) (at 39.37 22.8599 0)
+      (effects (font (size 1.27 1.27)) (justify left))
+    )
+    (property "Value" "MountingHole" (id 1) (at 39.37 25.3999 0)
+      (effects (font (size 1.27 1.27)) (justify left))
+    )
+    (property "Footprint" "MountingHole:MountingHole_4.3mm_M4" (id 2) (at 36.83 24.13 0)
+      (effects (font (size 1.27 1.27)) hide)
+    )
+    (property "Datasheet" "~" (id 3) (at 36.83 24.13 0)
+      (effects (font (size 1.27 1.27)) hide)
+    )
+  )
   (symbol (lib_id "power:PWR_FLAG") (at 46.99 81.28 270) (unit 1)
     (in_bom yes) (on_board yes) (fields_autoplaced)
@@
       (reference "F1") (unit 1) (value "xx mA") (footprint "0ESN_Lib:Fuse_1206_3216Metric_Pad1.42x1.75mm_HandSolder")
     )
+    (path "/3be81852-cc56-4f19-a97a-0a32a4554d57"
+      (reference "H1") (unit 1) (value "MountingHole") (footprint "MountingHole:MountingHole_4.3mm_M4")
+    )
+    (path "/2af81f78-b81a-48d1-80e8-b1fbb72a6951"
+      (reference "H2") (unit 1) (value "MountingHole") (footprint "MountingHole:MountingHole_4.3mm_M4")
+    )
+    (path "/35cfb696-d9fe-4ca4-84b3-89c00adcf94b"
+      (reference "H3") (unit 1) (value "MountingHole") (footprint "MountingHole:MountingHole_4.3mm_M4")
+    )
     (path "/74f97b6e-abd0-4c8d-a747-9bbde598ab0d"
