File: ModuleBattery18650.kicad_sch (KiCad schematic)
At the start: 31 parts, among them J1 Connector_2p, J2 Connector_2p_r, T1 SISH615ADN, T2 SISH615ADN, T3 FDN337N, T4 SISH615ADN, T5 SISH615ADN, U1 MCP121T-315E

Commit message: modification schema
Parts:
- removed D1: LED, Diode_SMD:D_0603_1608Metric_Pad1.05x0.95mm_HandSolder, symbol 0ESN_Lib:LED
- removed J1: Connector_2p, 0ESN_Lib:Connector_2p_m, symbol 0ESN_Lib:Connector_2p
- removed JP1: Jumper_2_Bridged, Jumper:SolderJumper-2_P1.3mm_Open_RoundedPad1.0x1.5mm, symbol 0ESN_Lib:Jumper_2_Bridged
- removed R1: 1M, Resistor_SMD:R_0603_1608Metric_Pad0.98x0.95mm_HandSolder, symbol Device:R
- removed R4: 150R, Resistor_SMD:R_0805_2012Metric_Pad1.20x1.40mm_HandSolder, symbol 0ESN_Lib:R
- removed RS1: 0R NP, Resistor_SMD:R_0603_1608Metric_Pad0.98x0.95mm_HandSolder, symbol Device:R
- removed T1, T2: SISH615ADN, 0ESN_Lib:PowerPAK 1212-8S, symbol 0ESN_Lib:SISH615ADN
- removed TP5, TP8: TestPoint, 0ESN_Lib:TestPoint_Pad_D1.0mm, symbol 0ESN_Lib:TestPoint
- added J1: Connector_3p, 0ESNLib:Connector_3p_m, symbol 0ESN_Lib:Connector_3p
- added JP1, JP2: SolderJumper_2_Bridged, Jumper:SolderJumper-2_P1.3mm_Open_RoundedPad1.0x1.5mm, symbol Jumper:SolderJumper_2_Bridged
- added TP4: TestPoint, 0ESN_Lib:TestPoint_Pad_D1.0mm, symbol 0ESN_Lib:TestPoint
- R1: renamed from R2; value 1M -> 100k
- R2: renamed from R3; value 1M -> 100k
- T1: renamed from T5; value SISH615ADN -> SISH101DN
- T2: renamed from T4; value SISH615ADN -> SISH101DN
- renumbered RS2 to RS1, TP4 to TP5, TP9 to TP8
Connections:
- net GND: now also J1.2 (P2)
- net Vbat: now also RS1.2, T2.5 (D); no longer T1.1 (S), T1.2 (S), T1.3 (S)
- net Vch: now also J1.1 (P1), JP1.1 (A)
- net at C1.1, F1.2: now also T1.5 (D), TP3.1, JP1.2 (B); no longer TP5.1
- net at R1.1, R2.1, RS1.1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: now also T1.1 (S), T1.2 (S), T1.3 (S), TP5.1
- net at R1.2, T3.1 (G), TP6.1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: now also JP2.2 (B), TP4.1
- new net: J1.3 (P3), JP2.1 (A)
Other:
- note added: "Reverse polarity protection"
- note added: "Using 2 P-Channel mosfet adds a serial resistor to the battery The SI2323DS has a Rds_on of about 39 mOhm with this voltage A better one like the SI7145DP has a Rds_on of up to 6 mOhm for 3V Or the SISH615ADN for a cheaper alternative, Rds_on up to 8 mOhm A serial resistance of 120 mOhm would mean that drawing 1 Amp from the current source, 120mW is dissiped into the mosfets"
- note added: "~{STATUS}"
- note removed: "Prevent reverse current"
- note removed: "Using 3 P-Channel mosfet adds a serial resistor to the battery The SI2323DS has a Rds_on of about 39 mOhm with this voltage A better one like the SI7145DP has a Rds_on of up to 6 mOhm for 3V Or the SISH615ADN for a cheaper alternative, Rds_on up to 8 mOhm A serial resistance of 120 mOhm would mean that drawing 1 Amp from the current source, 120mW is dissiped into the mosfets"
- note removed: "When over-discharge disabled : MCP121T consumes 1.75 uA R1 draws nothing R2 draws nothing R3 draws 3.08 uA Total is around 5 uA"
- note removed: "When over-discharge enabled : MCP121T consumes 1.75 uA R1 draws nothing R2 draws 3.08 uA (for 1 Mohm, need to verify that is enough to pull up T3) R3 draws nothing as the gate of T4 is High Total is around 5 uA"
- moved on the sheet: BT1, C1, F1, J2, R1, R2, RS1, T1, T2, T3, TP1, TP2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

Commit message: Version 3
Fixed schematic. Combined charge subcircuit disable and low voltage circuit cutoff
charge connector now 3pin
removed charge input reverse polarity protection
Parts:
- BT1: footprint 0ESN_Lib:18650_Battery_holder -> 0ESNLib:18650_Battery_holder
- F1: footprint 0ESN_Lib:Fuse_1206_3216Metric_Pad1.42x1.75mm_HandSolder -> 0ESNLib:Fuse_1206_3216Metric_Pad1.42x1.75mm_HandSolder
- J2: footprint 0ESN_Lib:Connector_2p_m -> 0ESNLib:Connector_2p_m
- T1, T2: footprint 0ESN_Lib:PowerPAK 1212-8S -> 0ESNLib:PowerPAK 1212-8S
- TP1, TP2, TP3, TP4, TP5, TP6, TP7, TP8: footprint 0ESN_Lib:TestPoint_Pad_D1.0mm -> 0ESNLib:TestPoint_Pad_D1.0mm
Connections:
- net at J1.3 (P3), JP2.1 (A): now also TP4.1
- net at JP2.2 (B), R1.2, T3.1 (G)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: no longer TP4.1
Other:
- moved on the sheet: TP4
Changed lines of the file:
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@@
   (junction (at 49.53 58.42) (diameter 0) (color 0 0 0 0)
   )
+  (junction (at 32.385 69.85) (diameter 0) (color 0 0 0 0)
+  )
   (junction (at 185.42 58.42) (diameter 0) (color 0 0 0 0)
   )
@@
   (junction (at 71.12 58.42) (diameter 0) (color 0 0 0 0)
   )
-  (junction (at 49.53 69.85) (diameter 0) (color 0 0 0 0)
-  )
   (junction (at 215.9 58.42) (diameter 0) (color 0 0 0 0)
   )
@@
     (stroke (width 0) (type default))
   )
+  (wire (pts (xy 32.385 69.85) (xy 38.735 69.85))
+    (stroke (width 0) (type default))
+  )
   (polyline (pts (xy 166.37 50.8) (xy 175.26 50.8))
     (stroke (width 0) (type default))
@@
     (stroke (width 0) (type default))
   )
-  (wire (pts (xy 49.53 69.85) (xy 55.88 69.85))
-    (stroke (width 0) (type default))
-  )
   (wire (pts (xy 156.21 58.42) (xy 163.83 58.42))
     (stroke (width 0) (type default))
@@
     (stroke (width 0) (type default))
   )
-  (wire (pts (xy 27.94 69.85) (xy 38.735 69.85))
+  (wire (pts (xy 27.94 69.85) (xy 32.385 69.85))
     (stroke (width 0) (type default))
   )
@@
     (effects (font (size 1.27 1.27)) (justify left bottom))
   )
+  (netclass_flag "" (length 2.54) (shape round) (at 59.055 58.42 0) (fields_autoplaced)
+    (effects (font (size 1.27 1.27)) (justify left bottom))
+    (property "Netclass" "Power" (at 59.7535 55.88 0)
+      (effects (font (size 1.27 1.27) italic) (justify left))
+    )
+  )
+  (netclass_flag "" (length 2.54) (shape round) (at 30.48 81.28 90) (fields_autoplaced)
+    (effects (font (size 1.27 1.27)) (justify left bottom))
+    (property "Netclass" "Power" (at 27.94 80.5815 90)
+      (effects (font (size 1.27 1.27) italic) (justify left))
+    )
+  )
+  (netclass_flag "" (length 2.54) (shape round) (at 182.88 68.58 270) (fields_autoplaced)
+    (effects (font (size 1.27 1.27)) (justify right bottom))
+    (property "Netclass" "Default" (at 185.42 67.8815 90)
+      (effects (font (size 1.27 1.27) italic) (justify left))
+    )
+  )
+  (netclass_flag "" (length 2.54) (shape round) (at 49.53 79.375 270) (fields_autoplaced)
+    (effects (font (size 1.27 1.27)) (justify right bottom))
+    (property "Netclass" "Default" (at 52.07 78.6765 90)
+      (effects (font (size 1.27 1.27) italic) (justify left))
+    )
+  )
+  (netclass_flag "" (length 2.54) (shape round) (at 83.82 69.85 90) (fields_autoplaced)
+    (effects (font (size 1.27 1.27)) (justify left bottom))
+    (property "Netclass" "Battery" (at 81.28 69.1515 90)
+      (effects (font (size 1.27 1.27) italic) (justify left))
+    )
+  )
+  (netclass_flag "" (length 2.54) (shape round) (at 32.385 58.42 180) (fields_autoplaced)
+    (effects (font (size 1.27 1.27)) (justify right bottom))
+    (property "Netclass" "Power" (at 33.0835 60.96 0)
+      (effects (font (size 1.27 1.27) italic) (justify left))
+    )
+  )
+  (netclass_flag "" (length 2.54) (shape round) (at 204.47 58.42 0) (fields_autoplaced)
+    (effects (font (size 1.27 1.27)) (justify left bottom))
+    (property "Netclass" "Power" (at 205.1685 55.88 0)
+      (effects (font (size 1.27 1.27) italic) (justify left))
+    )
+  )
+  (netclass_flag "" (length 2.54) (shape round) (at 32.385 69.85 180) (fields_autoplaced)
+    (effects (font (size 1.27 1.27)) (justify right bottom))
+    (property "Netclass" "Default" (at 33.0835 72.39 0)
+      (effects (font (size 1.27 1.27) italic) (justify left))
+    )
+  )
+  (netclass_flag "" (length 2.54) (shape round) (at 124.46 58.42 0) (fields_autoplaced)
+    (effects (font (size 1.27 1.27)) (justify left bottom))
+    (property "Netclass" "Power" (at 125.1585 55.88 0)
+      (effects (font (size 1.27 1.27) italic) (justify left))
+    )
+  )
   (symbol (lib_id "Device:Fuse") (at 83.82 64.77 180) (unit 1)
     (in_bom yes) (on_board yes) (dnp no) (fields_autoplaced)
@@
       (effects (font (size 1.27 1.27)) (justify right))
     )
-    (property "Footprint" "0ESN_Lib:Fuse_1206_3216Metric_Pad1.42x1.75mm_HandSolder" (at 85.598 64.77 90)
+    (property "Footprint" "0ESNLib:Fuse_1206_3216Metric_Pad1.42x1.75mm_HandSolder" (at 85.598 64.77 90)
       (effects (font (size 1.27 1.27)) hide)
     )
@@
       (effects (font (size 1.27 1.27)) hide)
     )
-    (property "Footprint" "0ESN_Lib:TestPoint_Pad_D1.0mm" (at 123.19 58.42 0)
+    (property "Footprint" "0ESNLib:TestPoint_Pad_D1.0mm" (at 123.19 58.42 0)
       (effects (font (size 1.27 1.27)) hide)
     )
@@
       (effects (font (size 1.27 1.27)) (justify left))
     )
-    (property "Footprint" "0ESN_Lib:18650_Battery_holder" (at 83.82 74.676 90)
+    (property "Footprint" "0ESNLib:18650_Battery_holder" (at 83.82 74.676 90)
       (effects (font (size 1.27 1.27)) hide)
     )
@@
       (effects (font (size 1.27 1.27)) hide)
     )
-    (property "Footprint" "0ESN_Lib:TestPoint_Pad_D1.0mm" (at 220.98 58.42 0)
+    (property "Footprint" "0ESNLib:TestPoint_Pad_D1.0mm" (at 220.98 58.42 0)
       (effects (font (size 1.27 1.27)) hide)
     )
@@
       (effects (font (size 1.27 1.27)) hide)
     )
-    (property "Footprint" "0ESN_Lib:TestPoint_Pad_D1.0mm" (at 30.48 82.55 0)
+    (property "Footprint" "0ESNLib:TestPoint_Pad_D1.0mm" (at 30.48 82.55 0)
       (effects (font (size 1.27 1.27)) hide)
     )
@@
       (effects (font (size 1.524 1.524)))
     )
-    (property "Footprint" "0ESN_Lib:PowerPAK 1212-8S" (at 102.87 59.055 0)
+    (property "Footprint" "0ESNLib:PowerPAK 1212-8S" (at 102.87 59.055 0)
       (effects (font (size 1.524 1.524)) hide)
     )
@@
       (effects (font (size 1.27 1.27)) hide)
     )
-    (property "Footprint" "0ESN_Lib:TestPoint_Pad_D1.0mm" (at 60.96 58.42 0)
+    (property "Footprint" "0ESNLib:TestPoint_Pad_D1.0mm" (at 60.96 58.42 0)
       (effects (font (size 1.27 1.27)) hide)
     )
@@
       (effects (font (size 1.27 1.27)) hide)
     )
-    (property "Footprint" "0ESN_Lib:TestPoint_Pad_D1.0mm" (at 165.1 80.01 0)
+    (property "Footprint" "0ESNLib:TestPoint_Pad_D1.0mm" (at 165.1 80.01 0)
       (effects (font (size 1.27 1.27)) hide)
     )
@@
     )
   )
-  (symbol (lib_id "0ESN_Lib:TestPoint") (at 55.88 69.85 0) (unit 1)
-    (in_bom yes) (on_board yes) (dnp no) (fields_autoplaced)
-    (property "Reference" "TP4" (at 55.88 64.77 0)
-      (effects (font (size 1.27 1.27)))
-    )
-    (property "Value" "TestPoint" (at 55.88 64.77 0)
-      (effects (font (size 1.27 1.27)) hide)
-    )
-    (property "Footprint" "0ESN_Lib:TestPoint_Pad_D1.0mm" (at 60.96 69.85 0)
-      (effects (font (size 1.27 1.27)) hide)
-    )
-    (property "Datasheet" "~" (at 60.96 69.85 0)
+  (symbol (lib_id "0ESN_Lib:TestPoint") (at 32.385 69.85 0) (unit 1)
+    (in_bom yes) (on_board yes) (dnp no) (fields_autoplaced)
+    (property "Reference" "TP4" (at 32.385 64.77 0)
+      (effects (font (size 1.27 1.27)))
+    )
+    (property "Value" "TestPoint" (at 32.385 64.77 0)
+      (effects (font (size 1.27 1.27)) hide)
+    )
+    (property "Footprint" "0ESNLib:TestPoint_Pad_D1.0mm" (at 37.465 69.85 0)
+      (effects (font (size 1.27 1.27)) hide)
+    )
+    (property "Datasheet" "~" (at 37.465 69.85 0)
       (effects (font (size 1.27 1.27)) hide)
     )
@@
       (effects (font (size 1.27 1.27)) hide)
     )
-    (property "Footprint" "0ESN_Lib:Connector_2p_m" (at 218.44 64.77 90)
+    (property "Footprint" "0ESNLib:Connector_2p_m" (at 218.44 64.77 90)
       (effects (font (size 1.27 1.27)) hide)
     )
@@
       (effects (font (size 1.27 1.27)) hide)
     )
-    (property "Footprint" "0ESN_Lib:TestPoint_Pad_D1.0mm" (at 187.96 68.58 0)
+    (property "Footprint" "0ESNLib:TestPoint_Pad_D1.0mm" (at 187.96 68.58 0)
       (effects (font (size 1.27 1.27)) hide)
     )
@@
       (effects (font (size 1.524 1.524)))
     )
-    (property "Footprint" "0ESN_Lib:PowerPAK 1212-8S" (at 173.99 59.055 0)
+    (property "Footprint" "0ESNLib:PowerPAK 1212-8S" (at 173.99 59.055 0)
       (effects (font (size 1.524 1.524)) hide)
     )
@@
       (effects (font (size 1.27 1.27)) hide)
     )
-    (property "Footprint" "0ESN_Lib:TestPoint_Pad_D1.0mm" (at 35.56 58.42 0)
-      (effects (font (size 1.27 1.27)) hide)
-    )
+    (property "Footprint" "0ESNLib:TestPoint_Pad_D1.0mm" (at 35.56 58.42 0)
+      (effects (font (size 1.27 1.27)) hide)
+    )
