File: ModuleBattery18650.kicad_pcb (KiCad board)
At the start: 2 copper layers, 83 x 30 mm, 31 parts, among them J1 Connector_2p, J2 Connector_2p_r, T1 SISH615ADN, T2 SISH615ADN, T3 FDN337N, T4 SISH615ADN, T5 SISH615ADN, U1 MCP121T-315E

Commit message: porte batterie adapté
Parts:
- BT1: footprint 0ESN_Lib:18650_Battery_holder -> 0ESNLib:18650_Battery_holder
Routing:
- net Net-(BT1-Pad1): track 20.7 -> 22.6 mm
Other:
- board text added: "TODO: 1. Vérifier l'espacement pour le porte batterie !!! Actuellement, le max n'est pas assez... Normalement ok 2. Vérifier si les connecteurs sont OK sur le montage actuel"
- board text removed: "TODO: 1. Vérifier l'espacement pour le porte batterie !!! Actuellement, le max n'est pas assez... 2. Vérifier si les connecteurs sont OK sur le montage actuel"
Changed lines of the file:
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@@
     )
   )
-  (footprint "0ESN_Lib:18650_Battery_holder" locked (layer "B.Cu")
+  (footprint "0ESNLib:18650_Battery_holder" (layer "B.Cu")
     (at 171.12 117.78)
     (property "Sheetfile" "ModuleBattery18650.kicad_sch")
     (property "Sheetname" "")
     (attr through_hole)
-    (fp_text reference "BT1" (at -21.7 6.35) (layer "B.SilkS")
+    (fp_text reference "BT1" (at -21.7 6.35 180) (layer "B.SilkS")
       (effects (font (size 1 1) (thickness 0.15)) (justify mirror))
     )
-    (fp_text value "LiIon 3.7V 4.2V" (at -21.7 8.89) (layer "B.Fab")
+    (fp_text value "LiIon 3.7V 4.2V" (at -21.7 8.89 180) (layer "B.Fab")
       (effects (font (size 1 1) (thickness 0.15)) (justify mirror))
     )
-    (fp_text user "+" (at -37.75 6.985) (layer "B.SilkS")
+    (fp_text user "+" (at -39.75 6.985 180) (layer "B.SilkS")
       (effects (font (size 2.032 2.032) (thickness 0.25)) (justify mirror))
     )
-    (fp_text user "-" (at -3.92 6.985 90) (layer "B.SilkS")
+    (fp_text user "-" (at -3.92 6.985 270) (layer "B.SilkS")
       (effects (font (size 2.032 2.032) (thickness 0.25)) (justify mirror))
     )
@@
       (effects (font (size 1 1) (thickness 0.15)))
     )
+    (fp_line (start 1.53 -5.08) (end -40.46 -5.08) (layer "B.SilkS") (width 0.15))
     (fp_line (start -40.46 5.08) (end 1.53 5.08) (layer "B.SilkS") (width 0.15))
-    (fp_line (start 1.53 -5.08) (end -40.46 -5.08) (layer "B.SilkS") (width 0.15))
     (fp_poly (pts
         (xy -2.396 5.08)
@@
         (xy -3.92 5.08)
       ) (layer "B.SilkS") (width 0.1) (fill solid))
+    (fp_line (start 15.13 5.08) (end -2.015 5.08) (layer "B.CrtYd") (width 0.12))
+    (fp_line (start -2.015 -5.08) (end 15.13 -5.08) (layer "B.CrtYd") (width 0.12))
+    (fp_line (start -54.895 -5.08) (end -42.83 -5.08) (layer "B.CrtYd") (width 0.12))
+    (fp_line (start 15.13 -5.08) (end 15.13 5.08) (layer "B.CrtYd") (width 0.12))
+    (fp_line (start -54.895 5.08) (end -54.895 -4.445) (layer "B.CrtYd") (width 0.12))
+    (fp_line (start -42.83 5.08) (end -54.895 5.08) (layer "B.CrtYd") (width 0.12))
+    (fp_line (start -54.895 -4.445) (end -54.895 -5.08) (layer "B.CrtYd") (width 0.12))
+    (fp_line (start -42.83 -5.08) (end -42.83 5.08) (layer "B.CrtYd") (width 0.12))
     (fp_line (start -2.015 5.08) (end -2.015 -5.08) (layer "B.CrtYd") (width 0.12))
-    (fp_line (start -40.83 -5.08) (end -40.83 5.08) (layer "B.CrtYd") (width 0.12))
-    (fp_line (start 15.13 5.08) (end -2.015 5.08) (layer "B.CrtYd") (width 0.12))
-    (fp_line (start 15.13 -5.08) (end 15.13 5.08) (layer "B.CrtYd") (width 0.12))
-    (fp_line (start -52.895 5.08) (end -52.895 -4.445) (layer "B.CrtYd") (width 0.12))
-    (fp_line (start -52.895 -4.445) (end -52.895 -5.08) (layer "B.CrtYd") (width 0.12))
-    (fp_line (start -52.895 -5.08) (end -40.83 -5.08) (layer "B.CrtYd") (width 0.12))
-    (fp_line (start -2.015 -5.08) (end 15.13 -5.08) (layer "B.CrtYd") (width 0.12))
-    (fp_line (start -40.83 5.08) (end -52.895 5.08) (layer "B.CrtYd") (width 0.12))
-    (fp_line (start -54 6.985) (end 15.13 6.985) (layer "B.Fab") (width 0.12))
-    (fp_line (start -54 -6.985) (end -54 6.985) (layer "B.Fab") (width 0.12))
+    (fp_line (start -56 6.985) (end 15.13 6.985) (layer "B.Fab") (width 0.12))
+    (fp_line (start 15.13 -6.985) (end -56 -6.985) (layer "B.Fab") (width 0.12))
     (fp_line (start 15.13 6.985) (end 15.13 -6.985) (layer "B.Fab") (width 0.12))
-    (fp_line (start 15.13 -6.985) (end -54 -6.985) (layer "B.Fab") (width 0.12))
-    (pad "1" thru_hole circle locked (at -50.62 0) (size 3.048 3.048) (drill 1.905) (layers *.Cu *.Mask)
+    (fp_line (start -56 -6.985) (end -56 6.985) (layer "B.Fab") (width 0.12))
+    (pad "1" thru_hole circle (at -45 -2.54) (size 3.048 3.048) (drill 1.905) (layers *.Cu *.Mask)
       (net 1 "Net-(BT1-Pad1)") (pinfunction "+") (pintype "passive"))
-    (pad "1" thru_hole circle locked (at -43 -2.54) (size 3.048 3.048) (drill 1.905) (layers *.Cu *.Mask)
+    (pad "1" thru_hole circle (at -52.62 0) (size 3.048 3.048) (drill 1.905) (layers *.Cu *.Mask)
       (net 1 "Net-(BT1-Pad1)") (pinfunction "+") (pintype "passive"))
-    (pad "1" thru_hole circle locked (at -43 2.54) (size 3.048 3.048) (drill 1.905) (layers *.Cu *.Mask)
+    (pad "1" thru_hole circle (at -45 2.54) (size 3.048 3.048) (drill 1.905) (layers *.Cu *.Mask)
       (net 1 "Net-(BT1-Pad1)") (pinfunction "+") (pintype "passive"))
-    (pad "2" thru_hole oval locked (at 9.739 0) (size 7.286 3.048) (drill oval 5 1.905) (layers *.Cu *.Mask)
+    (pad "2" thru_hole oval (at 9.739 0) (size 7.286 3.048) (drill oval 5 1.905) (layers *.Cu *.Mask)
       (net 2 "GND") (pinfunction "-") (pintype "passive"))
-    (pad "2" thru_hole oval locked (at 2.119 -2.54) (size 7.286 3.048) (drill oval 5 1.905) (layers *.Cu *.Mask)
+    (pad "2" thru_hole oval (at 2.119 2.54) (size 7.286 3.048) (drill oval 5 1.905) (layers *.Cu *.Mask)
       (net 2 "GND") (pinfunction "-") (pintype "passive"))
-    (pad "2" thru_hole oval locked (at 2.119 2.54) (size 7.286 3.048) (drill oval 5 1.905) (layers *.Cu *.Mask)
+    (pad "2" thru_hole oval (at 2.119 -2.54) (size 7.286 3.048) (drill oval 5 1.905) (layers *.Cu *.Mask)
       (net 2 "GND") (pinfunction "-") (pintype "passive"))
     (model "C:/Workspace/03_CAD_Output/Keystone_-_54.step"
@@
     (effects (font (size 1 1) (thickness 0.15)) (justify mirror))
   )
-  (gr_text "TODO:\n1. Vérifier l'espacement pour le porte batterie !!!\n   Actuellement, le max n'est pas assez...\n2. Vérifier si les connecteurs sont OK sur le montage actuel" (at 148.336 88.392) (layer "User.1")
+  (gr_text "TODO:\n1. Vérifier l'espacement pour le porte batterie !!!\n   Actuellement, le max n'est pas assez...\n	Normalement ok\n\n2. Vérifier si les connecteurs sont OK sur le montage actuel" (at 148.336 88.392) (layer "User.1")
     (effects (font (size 1.5 1.5) (thickness 0.3)))
   )
   (segment (start 134.0725 119.2675) (end 134.0725 117.78) (width 1.2) (layer "F.Cu") (net 1))
   (segment (start 133.02 120.32) (end 134.0725 119.2675) (width 1.2) (layer "F.Cu") (net 1))
-  (segment (start 128.12 120.32) (end 133.02 120.32) (width 1.2) (layer "F.Cu") (net 1))
-  (segment (start 120.5 117.78) (end 127.94 117.78) (width 1.2) (layer "B.Cu") (net 1))
-  (segment (start 128.12 117.6) (end 128.12 120.32) (width 1.2) (layer "B.Cu") (net 1))
-  (segment (start 128.12 115.24) (end 128.12 117.6) (width 1.2) (layer "B.Cu") (net 1))
-  (segment (start 127.94 117.78) (end 128.12 117.6) (width 1.2) (layer "B.Cu") (net 1))
+  (segment (start 126.12 120.32) (end 133.02 120.32) (width 1.2) (layer "F.Cu") (net 1))
+  (segment (start 126.06 117.78) (end 126.12 117.72) (width 1.2) (layer "B.Cu") (net 1))
+  (segment (start 118.5 117.78) (end 126.06 117.78) (width 1.2) (layer "B.Cu") (net 1))
+  (segment (start 126.12 115.24) (end 126.12 117.72) (width 1.2) (layer "B.Cu") (net 1))
+  (segment (start 126.12 117.72) (end 126.12 120.32) (width 1.2) (layer "B.Cu") (net 1))
   (segment (start 164.66 117.78) (end 164.66 119.05) (width 1.2) (layer "F.Cu") (net 2))
   (segment (start 139.1375 115.24) (end 139.1375 112.7215) (width 1.2) (layer "F.Cu") (net 2))

Commit message: Fixed portebatterie length
Parts:
- BT1: footprint 0ESNLib:18650_Battery_holder -> 0ESN_Lib:18650_Battery_holder
Routing:
- added copper zone on F.Cu, net GND
Other:
- board text added: "ModuleBattery18650 Nicolas Esseiva 2023.07.05 - r02"
- board text removed: "ModuleBattery18650 Nicolas Esseiva 2023.06.21 - r01"
- board text removed: "TODO: 1. Vérifier l'espacement pour le porte batterie !!! Actuellement, le max n'est pas assez... Normalement ok 2. Vérifier si les connecteurs sont OK sur le montage actuel"
Changed lines of the file:
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@@
       (svguseinch false)
       (svgprecision 6)
-      (excludeedgelayer false)
-      (plotframeref true)
+      (excludeedgelayer true)
+      (plotframeref false)
       (viasonmask false)
       (mode 1)
@@
       (sketchpadsonfab false)
       (subtractmaskfromsilk false)
-      (outputformat 4)
+      (outputformat 1)
       (mirror false)
       (drillshape 0)
       (scaleselection 1)
-      (outputdirectory "fabrication/pdf")
+      (outputdirectory "fabrication/gerber")
     )
   )
@@
     )
   )
-  (footprint "0ESNLib:18650_Battery_holder" (layer "B.Cu")
+  (footprint "0ESN_Lib:18650_Battery_holder" (layer "B.Cu")
     (at 171.12 117.78)
     (property "Sheetfile" "ModuleBattery18650.kicad_sch")
@@
     )
     (fp_line (start 1.53 -5.08) (end -40.46 -5.08) (layer "B.SilkS") (width 0.15))
+    (fp_line (start 1 6.95) (end 2.05 6.95) (layer "B.SilkS") (width 0.1))
+    (fp_line (start 2.975 6.95) (end 4.025 6.95) (layer "B.SilkS") (width 0.1))
+    (fp_line (start 0.975 6.05) (end 2.025 6.05) (layer "B.SilkS") (width 0.1))
     (fp_line (start -40.46 5.08) (end 1.53 5.08) (layer "B.SilkS") (width 0.15))
+    (fp_line (start 2.95 6.05) (end 4 6.05) (layer "B.SilkS") (width 0.1))
+    (fp_rect (start 2 6) (end 3 7) (layer "B.SilkS") (width 0) (fill solid))
+    (fp_rect (start 4 6) (end 5 7) (layer "B.SilkS") (width 0) (fill solid))
+    (fp_rect (start 0 6) (end 1 7) (layer "B.SilkS") (width 0) (fill solid))
     (fp_poly (pts
         (xy -2.396 5.08)
@@
         (xy -3.92 5.08)
       ) (layer "B.SilkS") (width 0.1) (fill solid))
+    (fp_line (start -2.015 -5.08) (end 15.13 -5.08) (layer "B.CrtYd") (width 0.12))
+    (fp_line (start -54.895 -4.445) (end -54.895 -5.08) (layer "B.CrtYd") (width 0.12))
+    (fp_line (start 15.13 -5.08) (end 15.13 5.08) (layer "B.CrtYd") (width 0.12))
+    (fp_line (start -54.895 -5.08) (end -42.83 -5.08) (layer "B.CrtYd") (width 0.12))
+    (fp_line (start -42.83 -5.08) (end -42.83 5.08) (layer "B.CrtYd") (width 0.12))
     (fp_line (start 15.13 5.08) (end -2.015 5.08) (layer "B.CrtYd") (width 0.12))
-    (fp_line (start -2.015 -5.08) (end 15.13 -5.08) (layer "B.CrtYd") (width 0.12))
-    (fp_line (start -54.895 -5.08) (end -42.83 -5.08) (layer "B.CrtYd") (width 0.12))
-    (fp_line (start 15.13 -5.08) (end 15.13 5.08) (layer "B.CrtYd") (width 0.12))
     (fp_line (start -54.895 5.08) (end -54.895 -4.445) (layer "B.CrtYd") (width 0.12))
+    (fp_line (start -2.015 5.08) (end -2.015 -5.08) (layer "B.CrtYd") (width 0.12))
     (fp_line (start -42.83 5.08) (end -54.895 5.08) (layer "B.CrtYd") (width 0.12))
-    (fp_line (start -54.895 -4.445) (end -54.895 -5.08) (layer "B.CrtYd") (width 0.12))
-    (fp_line (start -42.83 -5.08) (end -42.83 5.08) (layer "B.CrtYd") (width 0.12))
-    (fp_line (start -2.015 5.08) (end -2.015 -5.08) (layer "B.CrtYd") (width 0.12))
+    (fp_line (start -56 -6.985) (end -56 6.985) (layer "B.Fab") (width 0.12))
     (fp_line (start -56 6.985) (end 15.13 6.985) (layer "B.Fab") (width 0.12))
+    (fp_line (start 15.13 6.985) (end 15.13 -6.985) (layer "B.Fab") (width 0.12))
     (fp_line (start 15.13 -6.985) (end -56 -6.985) (layer "B.Fab") (width 0.12))
-    (fp_line (start 15.13 6.985) (end 15.13 -6.985) (layer "B.Fab") (width 0.12))
-    (fp_line (start -56 -6.985) (end -56 6.985) (layer "B.Fab") (width 0.12))
+    (pad "1" thru_hole circle (at -52.62 0) (size 3.048 3.048) (drill 1.905) (layers *.Cu *.Mask)
+      (net 1 "Net-(BT1-Pad1)") (pinfunction "+") (pintype "passive"))
     (pad "1" thru_hole circle (at -45 -2.54) (size 3.048 3.048) (drill 1.905) (layers *.Cu *.Mask)
-      (net 1 "Net-(BT1-Pad1)") (pinfunction "+") (pintype "passive"))
-    (pad "1" thru_hole circle (at -52.62 0) (size 3.048 3.048) (drill 1.905) (layers *.Cu *.Mask)
       (net 1 "Net-(BT1-Pad1)") (pinfunction "+") (pintype "passive"))
     (pad "1" thru_hole circle (at -45 2.54) (size 3.048 3.048) (drill 1.905) (layers *.Cu *.Mask)
       (net 1 "Net-(BT1-Pad1)") (pinfunction "+") (pintype "passive"))
-    (pad "2" thru_hole oval (at 9.739 0) (size 7.286 3.048) (drill oval 5 1.905) (layers *.Cu *.Mask)
+    (pad "2" thru_hole oval (at 2.5 2.54) (size 8.048 3.048) (drill oval 6.905 1.905) (layers *.Cu *.Mask)
       (net 2 "GND") (pinfunction "-") (pintype "passive"))
-    (pad "2" thru_hole oval (at 2.119 2.54) (size 7.286 3.048) (drill oval 5 1.905) (layers *.Cu *.Mask)
+    (pad "2" thru_hole oval (at 2.5 -2.54) (size 8.048 3.048) (drill oval 6.905 1.905) (layers *.Cu *.Mask)
       (net 2 "GND") (pinfunction "-") (pintype "passive"))
-    (pad "2" thru_hole oval (at 2.119 -2.54) (size 7.286 3.048) (drill oval 5 1.905) (layers *.Cu *.Mask)
+    (pad "2" thru_hole oval (at 10.12 0) (size 8.048 3.048) (drill oval 6.905 1.905) (layers *.Cu *.Mask)
       (net 2 "GND") (pinfunction "-") (pintype "passive"))
     (model "C:/Workspace/03_CAD_Output/Keystone_-_54.step"
@@
     (effects (font (size 1 1) (thickness 0.15)) (justify mirror))
   )
-  (gr_text "ModuleBattery18650\nNicolas Esseiva\n2023.06.21 - r01" (at 125.73 107.95 180) (layer "B.SilkS")
+  (gr_text "ModuleBattery18650\nNicolas Esseiva\n2023.07.05 - r02" (at 125.73 107.95 180) (layer "B.SilkS")
     (effects (font (size 1.27 1.27) (thickness 0.3)) (justify mirror))
   )
   (gr_text "CHARGE" (at 132.715 100.965 270) (layer "B.SilkS")
     (effects (font (size 1 1) (thickness 0.15)) (justify mirror))
-  )
-  (gr_text "TODO:\n1. Vérifier l'espacement pour le porte batterie !!!\n   Actuellement, le max n'est pas assez...\n	Normalement ok\n\n2. Vérifier si les connecteurs sont OK sur le montage actuel" (at 148.336 88.392) (layer "User.1")
-    (effects (font (size 1.5 1.5) (thickness 0.3)))
   )
   (segment (start 134.0725 119.2675) (end 134.0725 117.78) (width 1.2) (layer "F.Cu") (net 1))
@@
   (segment (start 145.72 121.844) (end 139.37 121.844) (width 1.2) (layer "B.Cu") (net 2))
   (segment (start 137.084 112.7) (end 143.688 112.7) (width 1.2) (layer "B.Cu") (net 2))
-  (segment (start 172.87 117.808) (end 172.87 120.32) (width 1.2) (layer "B.Cu") (net 2))
   (segment (start 156.278 120.574) (end 156.278 121.7) (width 1.2) (layer "B.Cu") (net 2))
   (segment (start 137.084 113.606) (end 137.084 118.796) (width 1.2) (layer "B.Cu") (net 2))
@@
   (segment (start 136.9144 113.4364) (end 137.084 113.606) (width 0.5) (layer "B.Cu") (net 2))
   (segment (start 146.118 120.828) (end 146.118 121.844) (width 1.2) (layer "B.Cu") (net 2))
-  (segment (start 172.898 117.78) (end 172.87 117.808) (width 1.2) (layer "B.Cu") (net 2))
   (segment (start 166.6748 113.0046) (end 166.802 112.8774) (width 0.5) (layer "B.Cu") (net 2))
   (segment (start 157.658 121.844) (end 156.134 121.844) (width 1.2) (layer "B.Cu") (net 2))
-  (segment (start 172.87 115.24) (end 172.87 117.808) (width 1.2) (layer "B.Cu") (net 2))
   (segment (start 156.278 121.7) (end 156.134 121.844) (width 1.2) (layer "B.Cu") (net 2))
   (segment (start 137.084 118.796) (end 137.084 119.558) (width 1.2) (layer "B.Cu") (net 2))
   (segment (start 139.1375 101.0375) (end 138.43 100.33) (width 1.2) (layer "B.Cu") (net 2))
   (segment (start 126.1655 105.2105) (end 139.1375 105.2105) (width 0.5) (layer "B.Cu") (net 2))
+  (segment (start 173.62 115.24) (end 173.62 120.32) (width 1.2) (layer "B.Cu") (net 2))
   (segment (start 138.43 100.33) (end 137.16 100.33) (width 1.2) (layer "B.Cu") (net 2))
   (segment (start 141.91 122.225) (end 141.91 120.4235) (width 0.5) (layer "F.Cu") (net 3))
@@
   (segment (start 150.8 123.114) (end 150.8 121.844) (width 0.25) (layer "F.Cu") (net 11))
   (segment (start 149.1725 118.7825) (end 149.21 118.82) (width 0.25) (layer "F.Cu") (net 11))
-  (zone (net 2) (net_name "GND") (layer "B.Cu") (hatch edge 0.508)
+  (zone (net 2) (net_name "GND") (layers F&B.Cu) (hatch edge 0.508)
     (connect_pads (clearance 0.17))
     (min_thickness 0.254) (filled_areas_thickness no)

Commit message: modification schema
Parts:
- removed D1: LED, Diode_SMD:D_0603_1608Metric_Pad1.05x0.95mm_HandSolder
- removed R3: 1M, Resistor_SMD:R_0603_1608Metric_Pad0.98x0.95mm_HandSolder
- removed R4: 150R, Resistor_SMD:R_0805_2012Metric_Pad1.20x1.40mm_HandSolder
- removed RS2: 0R NP, Resistor_SMD:R_0603_1608Metric_Pad0.98x0.95mm_HandSolder
- removed T4, T5: SISH615ADN, 0ESN_Lib:PowerPAK 1212-8S
- removed TP9: TestPoint, 0ESN_Lib:TestPoint_Pad_D1.0mm
- added JP2: SolderJumper_2_Bridged, Jumper:SolderJumper-2_P1.3mm_Open_RoundedPad1.0x1.5mm, F.Cu at (137.8, 91.4)
- J1: value Connector_2p -> Connector_3p; footprint 0ESN_Lib:Connector_2p_m -> 0ESNLib:Connector_3p_m
- JP1: value Jumper_2_Bridged -> SolderJumper_2_Bridged
- R1, R2: value 1M -> 100k
- T1, T2: value SISH615ADN -> SISH101DN
- moved J1 2.56 mm to (137.2, 105.4)
Connections:
- C1 pad 1: Net-(C1-Pad1) -> Net-(JP1-B)
- F1 pad 2: Net-(C1-Pad1) -> Net-(JP1-B)
- JP1 pad 2: Net-(D1-Pad1) -> Net-(JP1-B)
- R1 pad 1: Net-(D1-Pad1) -> Net-(U1-VDD)
- R1 pad 2: GND -> Net-(JP2-B)
- R2 pad 1: Net-(R2-Pad1) -> Net-(U1-VDD)
- R2 pad 2: Net-(R2-Pad2) -> Net-(T2-G)
- RS1 pad 1: Net-(C1-Pad1) -> Net-(U1-VDD)
- RS1 pad 2: Net-(R2-Pad1) -> /Vbat
- T1 pad 1: Net-(C1-Pad1) -> Net-(U1-VDD)
- T1 pad 2: Net-(C1-Pad1) -> Net-(U1-VDD)
- T1 pad 3: Net-(C1-Pad1) -> Net-(U1-VDD)
- T1 pad 5: Net-(D1-Pad1) -> Net-(JP1-B)
- T2 pad 1: Net-(C1-Pad1) -> Net-(U1-VDD)
- T2 pad 2: Net-(C1-Pad1) -> Net-(U1-VDD)
- T2 pad 3: Net-(C1-Pad1) -> Net-(U1-VDD)
- T2 pad 4: Net-(D1-Pad1) -> Net-(T2-G)
- T2 pad 5: Net-(R2-Pad1) -> /Vbat
- T3 pad 1: Net-(R2-Pad2) -> Net-(JP2-B)
- T3 pad 3: Net-(R3-Pad2) -> Net-(T2-G)
- TP3 pad 1: Net-(D1-Pad1) -> Net-(JP1-B)
- TP4 pad 1: Net-(C1-Pad1) -> Net-(JP2-B)
- TP5 pad 1: Net-(R2-Pad1) -> Net-(U1-VDD)
- TP6 pad 1: Net-(R2-Pad2) -> Net-(JP2-B)
- TP7 pad 1: Net-(R3-Pad2) -> Net-(T2-G)
- TP8 pad 1: Net-(RS2-Pad2) -> /Vbat
- U1 pad 1: Net-(R2-Pad2) -> Net-(JP2-B)
- U1 pad 2: Net-(R2-Pad1) -> Net-(U1-VDD)
Routing:
- net (no net): track 0.00 -> 121.9 mm, vias 0 -> 3
- net Net-(D1-Pad1): track 39.5 -> 0.00 mm, vias 3 -> 0
- net Net-(R2-Pad1): track 38.0 -> 0.00 mm, vias 2 -> 0
- net Net-(C1-Pad1): track 32.9 -> 0.00 mm
- net Net-(RS2-Pad2): track 28.8 -> 0.00 mm
- net /Vbat: track 24.3 -> 53.1 mm
- net Net-(T2-G): track 0.00 -> 13.2 mm, vias 0 -> 2
- net Net-(R3-Pad2): track 13.2 -> 0.00 mm, vias 2 -> 0
- net Net-(R2-Pad2): track 9.53 -> 0.00 mm
- net Net-(D1-Pad2): track 1.96 -> 0.00 mm
- net Net-(U1-VDD): vias 0 -> 2
